Commit message: updates

File: src/my_robot/urdf/my_robot.xacro (robot description, xacro)
@@ -57,5 +57,5 @@
                                                   </link>
   <joint type="continuous" name="right_wheel_hinge">
-    <origin xyz="0 0.13 0" rpy="0 0 0"/>
+    <origin xyz="0 -0.13 0" rpy="0 0 0"/>
     <child link="right_wheel"/>
     <parent link="chassis"/>
@@ -72,5 +72,5 @@
     </visual>
     <collision>
-      <origin xyz="0.0 0.0 0.0" rpy="0.0 1.5707 0.0"/>
+      <origin xyz="0.0 0.0 0.0" rpy="0.0 1.5707 1.5707"/>
       <geometry>
         <cylinder length="0.05" radius="0.1"/>
@@ -88,5 +88,5 @@
   </link>
   <joint type="continuous" name="left_wheel_hinge">
-    <origin xyz="0 -0.13 0" rpy="0 0 0"/>
+    <origin xyz="0 0.13 0" rpy="0 0 0"/>
     <child link="left_wheel"/>
     <parent link="chassis"/>
@@ -189,3 +189,6 @@
     <material>Gazebo/Green</material>
 </gazebo>
+<gazebo reference="right_wheel">
+    <material>Gazebo/Red</material>
+</gazebo>
 </robot>

Commit message: removed sleep file per feedback

File: src/my_robot/urdf/my_robot.xacro (robot description, xacro)
@@ -28,9 +28,9 @@
                                                       <origin xyz="0 0 0.1" rpy=" 0 0 0"/>
                                                       <geometry>
-                                                        <box size=".4 .2 .2"/>
+                                                        <box size=".4 .2 .4"/>
                                                       </geometry>
                                                     </visual>
                                                     <collision name='back_caster_collision'>
-                                                      <origin xyz="-0.15 0 -0.05" rpy=" 0 0 0"/>
+                                                      <origin xyz="-0.15 0 -0.15" rpy=" 0 0 0"/>
                                                       <geometry>
                                                         <sphere radius="0.0499"/>
@@ -38,5 +38,5 @@
                                                     </collision>
                                                     <visual name='back_caster_visual'>
-                                                      <origin xyz="-0.15 0 -0.05" rpy=" 0 0 0"/>
+                                                      <origin xyz="-0.15 0 -0.15" rpy=" 0 0 0"/>
                                                       <geometry>
                                                         <sphere radius="0.05"/>
@@ -44,5 +44,5 @@
                                                     </visual>
                                                     <collision name='front_caster_collision'>
-                                                      <origin xyz="0.15 0 -0.05" rpy=" 0 0 0"/>
+                                                      <origin xyz="0.15 0 -0.15" rpy=" 0 0 0"/>
                                                       <geometry>
                                                         <sphere radius="0.0499"/>
@@ -50,5 +50,5 @@
                                                     </collision>
                                                     <visual name='front_caster_visual'>
-                                                      <origin xyz="0.15 0 -0.05" rpy=" 0 0 0"/>
+                                                      <origin xyz="0.15 0 -0.15" rpy=" 0 0 0"/>
                                                       <geometry>
                                                         <sphere radius="0.05"/>
@@ -68,5 +68,5 @@
       <origin xyz="0.0 0.0 0.0" rpy="0 1.5707 1.5707"/>
       <geometry>
-        <cylinder length="0.05" radius="0.1"/>
+        <cylinder length="0.05" radius="0.2"/>
       </geometry>
     </visual>
@@ -74,5 +74,5 @@
       <origin xyz="0.0 0.0 0.0" rpy="0.0 1.5707 1.5707"/>
       <geometry>
-        <cylinder length="0.05" radius="0.1"/>
+        <cylinder length="0.05" radius="0.2"/>
       </geometry>
     </collision>
@@ -99,5 +99,5 @@
       <origin xyz="0.0 0.0 0.0" rpy="0 01.5707 1.5707"/>
       <geometry>
-        <cylinder length="0.05" radius="0.1"/>
+        <cylinder length="0.05" radius="0.2"/>
       </geometry>
     </visual>
@@ -105,5 +105,5 @@
       <origin xyz="0.0 0.0 0.0" rpy="0.0 1.5707 1.5707"/>
       <geometry>
-        <cylinder length="0.05" radius="0.1"/>
+        <cylinder length="0.05" radius="0.2"/>
       </geometry>
     </collision>
@@ -153,5 +153,5 @@
   </link>
   <joint type="fixed" name="hokuyo_joint">
-    <origin xyz="0.15 0 0.1" rpy="0 0 0"/>
+    <origin xyz="0.15 0 0.22" rpy="0 0 0"/>
     <child link="hokuyo"/>
     <parent link="chassis"/>
